File: Hardware/Vitalung_V0.1/Vitalung_V0.1.kicad_pcb (KiCad board)
At the start: 2 copper layers, 80 x 22 mm, 52 parts, among them J1 Conn_01x06, Q1 FS8205A, Q2 AO3400A, Q3 AO3401A, SW1 SW_SPDT, U1 ESP32C3_Seeed-Studio, U10 MT3608, U2 DW01A, U3 TP5100, U4 AMS1117-3.3

Commit message: PCB changes
Parts:
- added H1: MountingHole, MountingHole:MountingHole_2.2mm_M2, F.Cu at (121.8, 85.0)
- added H2: MountingHole, MountingHole:MountingHole_2.2mm_M2, F.Cu at (196.0, 113.0)
Other:
- board size 80 x 22 mm -> 82.2 x 36 mm

Commit message: PCB DXF change
Parts:
- removed Q3: AO3401A, Package_TO_SOT_SMD:SOT-23
- removed R14: 100K, Resistor_SMD:R_0603_1608Metric_Pad0.98x0.95mm_HandSolder
- added H3: MountingHole, MountingHole:MountingHole_2.2mm_M2, F.Cu at (120.8, 107.0)
- added H4: MountingHole, MountingHole:MountingHole_2.2mm_M2, F.Cu at (194.8, 80.0)
- SW1: footprint Button_Switch_SMD:SW_SPDT_PCM12 -> Button_Switch_THT:SW_Slide_SPDT_Angled_CK_OS102011MA1Q
- moved SW1 11.7 mm to (159.8, 79.5)
- moved D2 11.2 mm to (187.8, 81.0)
- moved U1 11.1 mm to (165.6, 98.2)
- moved C15 11.0 mm to (185.8, 80.2)
- moved C14 10.9 mm to (185.7, 84.3)
- moved R13 10.8 mm to (189.1, 85.7)
- moved R3 10.4 mm to (162.5, 91.8)
- moved R4 10.3 mm to (162.5, 93.9)
- moved D1 10.0 mm to (147.3, 81.0)
- moved R6 8.25 mm to (163.5, 84.3)
- moved C13 8.15 mm to (161.5, 88.4)
- moved R7 8.15 mm to (163.5, 88.4)
- moved H2 6.12 mm to (194.8, 107.0)
- moved R5 5.69 mm to (144.8, 86.4)
- moved TP2 5.58 mm to (137.9, 84.8)
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Connections:
- C17 pad 1: Net-(Q3-D) -> Net-(SW1-A)
- L1 pad 1: Net-(Q3-D) -> Net-(SW1-A)
- R13 pad 1: Net-(U1-PA02_A0_D0) -> Net-(U1-PA10_A2_D2)
- R6 pad 2: Net-(Q3-D) -> Net-(SW1-A)
- SW1 pad 1: Net-(Q3-G) -> Net-(SW1-A)
- SW1 pad 2: GND -> +BATT
- U1 pad 1: Net-(U1-PA02_A0_D0) -> unconnected-(U1-PA02_A0_D0-Pad1)
- U1 pad 3: unconnected-(U1-PA10_A2_D2-Pad3) -> Net-(U1-PA10_A2_D2)
- U1 pad 4: Heater_En -> unconnected-(U1-PA11_A3_D3-Pad4)
- U1 pad 7: unconnected-(U1-PB08_A6_D6_TX-Pad7) -> Heater_En
- U10 pad 4: Net-(Q3-D) -> Net-(SW1-A)
- U10 pad 5: Net-(Q3-D) -> Net-(SW1-A)
Routing:
- net Net-(U1-PA02_A0_D0): track 26.8 -> 0.00 mm, vias 2 -> 0
- net Net-(U1-PA10_A2_D2): track 0.00 -> 26.4 mm, vias 0 -> 2
- net Net-(SW1-A): track 0.00 -> 23.7 mm
- net Net-(Q3-D): track 15.4 -> 0.00 mm
- net SDA: track 10.9 -> 25.6 mm, vias 1 -> 0
- net SCL: track 16.7 -> 26.3 mm, vias 1 -> 0
- net +5V: track 65.8 -> 75.3 mm
- net Net-(Q3-G): track 9.24 -> 0.00 mm, vias 2 -> 0
- net Net-(D1-K2): track 16.6 -> 21.4 mm, vias 1 -> 2
- net Net-(D1-K1): track 19.2 -> 24.0 mm, vias 1 -> 2
- net +3V3: track 55.9 -> 60.3 mm
- net VBUS: track 76.8 -> 73.4 mm
- net Net-(BT1--): track 78.3 -> 76.1 mm
- net Net-(J1-Pin_1): track 6.65 -> 8.56 mm
- net +BATT: track 60.1 -> 58.8 mm, vias 2 -> 1
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Other:
- board size 82.2 x 36 mm -> 80 x 33 mm

Commit message: Gerber generation
Connections:
- net Net-(D1-K1) renamed /Red
- net Net-(D1-K2) renamed /Green
Other:
- board text added: "+"
- board text added: "Green"
- board text added: "Red"
- board text added: "Vitalung_V0.1"
Changed lines of the file:
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@@
 	)
 	(paper "A4")
+	(title_block
+		(title "Vitalung")
+		(date "2026-02-05")
+		(rev "0.1")
+	)
 	(layers
 		(0 "F.Cu" signal)
@@
 			(plotframeref no)
 			(mode 1)
-			(useauxorigin no)
+			(useauxorigin yes)
 			(hpglpennumber 1)
 			(hpglpenspeed 20)
@@
 			(outputformat 1)
 			(mirror no)
-			(drillshape 1)
+			(drillshape 0)
 			(scaleselection 1)
-			(outputdirectory "")
+			(outputdirectory "D:/Github/Vitalung/Hardware/Vitalung_V0.1/Gerber_Vitalung_V0.1/")
 		)
 	)
@@
 	(net 30 "unconnected-(U2-TD-Pad4)")
 	(net 31 "unconnected-(U10-NC-Pad6)")
-	(net 32 "Net-(D1-K2)")
-	(net 33 "Net-(D1-K1)")
+	(net 32 "/Green")
+	(net 33 "/Red")
 	(net 34 "unconnected-(SW1-C-Pad3)")
 	(net 35 "Net-(D2-A)")
@@
 		(sheetname "/")
 		(sheetfile "Vitalung_V0.1.kicad_sch")
-		(attr exclude_from_pos_files)
+		(attr exclude_from_pos_files exclude_from_bom)
 		(fp_circle
 			(center 0 0)
@@
 			)
 		)
-		(property "Robu_SKU" "R181035"
+		(property "Robu_SKU" ""
 			(at 0 0 180)
 			(unlocked yes)
@@
 		(sheetname "/")
 		(sheetfile "Vitalung_V0.1.kicad_sch")
-		(attr exclude_from_pos_files)
+		(attr exclude_from_pos_files exclude_from_bom)
 		(fp_circle
 			(center 0 0)
@@
 		(sheetname "/")
 		(sheetfile "Vitalung_V0.1.kicad_sch")
-		(attr exclude_from_pos_files)
+		(attr exclude_from_pos_files exclude_from_bom)
 		(fp_circle
 			(center 0 0)
@@
 		(sheetname "/")
 		(sheetfile "Vitalung_V0.1.kicad_sch")
-		(attr exclude_from_pos_files)
+		(attr exclude_from_pos_files exclude_from_bom)
 		(fp_circle
 			(center 0 0)
@@
 			(layers "*.Cu" "*.Mask")
 			(remove_unused_layers no)
-			(net 33 "Net-(D1-K1)")
+			(net 33 "/Red")
 			(pinfunction "K1")
 			(pintype "input")
@@
 			(layers "*.Cu" "*.Mask")
 			(remove_unused_layers no)
-			(net 32 "Net-(D1-K2)")
+			(net 32 "/Green")
 			(pinfunction "K2")
 			(pintype "input")
@@
 		(sheetname "/")
 		(sheetfile "Vitalung_V0.1.kicad_sch")
-		(attr exclude_from_pos_files)
+		(attr exclude_from_pos_files exclude_from_bom)
 		(fp_circle
 			(center 0 0)
@@
 			(layers "F.Cu" "F.Mask" "F.Paste")
 			(roundrect_rratio 0.25)
-			(net 32 "Net-(D1-K2)")
+			(net 32 "/Green")
 			(pinfunction "~{STDBY}")
 			(pintype "passive")
@@
 			(layers "F.Cu" "F.Mask" "F.Paste")
 			(roundrect_rratio 0.25)
-			(net 33 "Net-(D1-K1)")
+			(net 33 "/Red")
 			(pinfunction "~{CHRG}")
 			(pintype "passive")
@@
 		(layer "Edge.Cuts")
 	)
+	(gr_text "Red"
+		(at 146.1 79.4 0)
+		(layer "F.SilkS")
+		(effects
+			(font
+				(size 1.5 1.5)
+				(thickness 0.3)
+				(bold yes)
+			)
+			(justify left bottom)
+		)
+	)
+	(gr_text "+"
+		(at 189.5 79.1 0)
+		(layer "F.SilkS")
+		(effects
+			(font
+				(size 1.5 1.5)
+				(thickness 0.3)
+				(bold yes)
+			)
+			(justify left bottom)
+		)
+	)
+	(gr_text "Green"
+		(at 136.6 79.4 0)
+		(layer "F.SilkS")
+		(effects
+			(font
+				(size 1.5 1.5)
+				(thickness 0.3)
+				(bold yes)
+			)
+			(justify left bottom)
+		)
+	)
+	(gr_text "Vitalung_V0.1"
+		(at 126 109.2 0)
+		(layer "F.SilkS")
+		(effects
+			(font
+				(size 1.5 1.5)
+				(thickness 0.3)
+				(bold yes)
+			)
+			(justify left bottom)
+		)
+	)
 	(segment
