File: Hardware/Vitalung_V0.1/Vitalung_V0.1.kicad_sch (KiCad schematic)
At the start: 1 part, among them U1 ESP32C3_Seeed-Studio

Commit message: PCB completion
Parts:
- added BT1: Battery_Cell, Battery:BatteryHolder_MPD_BH-18650-PC2, symbol Device:Battery_Cell
- added C1, C10, C13, C14, C15, C4, C5: 100nF, Capacitor_SMD:C_0603_1608Metric_Pad1.08x0.95mm_HandSolder, symbol Device:C_Small
- added C11, C12, C17, C18, C3, C6, C9: 10uF, Capacitor_SMD:C_0805_2012Metric_Pad1.18x1.45mm_HandSolder, symbol Device:C_Small
- added D1: LED_Dual_KAK, LED_THT:LED_D3.0mm-3, symbol Device:LED_Dual_KAK
- added D2: LED, LED_THT:LED_D3.0mm, symbol Device:LED_Small
- added D3: SMAJ5.0A, Diode_SMD:D_SMA, symbol Diode:SMAJ5.0A
- added D4: SS34, Diode_SMD:D_SMA, symbol Device:D_Schottky_Small
- added J1: Conn_01x06, Connector_PinHeader_2.54mm:PinHeader_1x06_P2.54mm_Vertical, symbol Connector_Generic:Conn_01x06
- added L1: 4.7uH, Inductor_SMD:L_Abracon_ASPI-0425, symbol Device:L_Small
- added L2: 22uH, Inductor_SMD:L_Abracon_ASPI-0630LR, symbol Device:L_Small
- added Q1: FS8205A, Package_TO_SOT_SMD:SOT-23-6, symbol Transistor_FET:DMG9926UDM
- added Q2: AO3400A, Package_TO_SOT_SMD:SOT-23, symbol Transistor_FET:AO3400A
- added Q3: AO3401A, Package_TO_SOT_SMD:SOT-23, symbol Transistor_FET:AO3401A
- added R1: 100R, Resistor_SMD:R_0603_1608Metric_Pad0.98x0.95mm_HandSolder, symbol Device:R_Small
- added R10, R2, R5: 1K, Resistor_SMD:R_0603_1608Metric_Pad0.98x0.95mm_HandSolder, symbol Device:R_Small
- added R11, R3, R4: 10K, Resistor_SMD:R_0603_1608Metric_Pad0.98x0.95mm_HandSolder, symbol Device:R_Small
- added R12: 0R, Resistor_SMD:R_0603_1608Metric_Pad0.98x0.95mm_HandSolder, symbol Device:R_Small
- added R13: 470R, Resistor_SMD:R_0603_1608Metric_Pad0.98x0.95mm_HandSolder, symbol Device:R_Small
- added R14, R6: 100K, Resistor_SMD:R_0603_1608Metric_Pad0.98x0.95mm_HandSolder, symbol Device:R_Small
- added R18: 20K, Resistor_SMD:R_0603_1608Metric_Pad0.98x0.95mm_HandSolder, symbol Device:R_Small
- added R19: 2.7K, Resistor_SMD:R_0603_1608Metric_Pad0.98x0.95mm_HandSolder, symbol Device:R_Small
- added R7: 180K, Resistor_SMD:R_0603_1608Metric_Pad0.98x0.95mm_HandSolder, symbol Device:R_Small
- added R8: TBD, Resistor_SMD:R_0603_1608Metric_Pad0.98x0.95mm_HandSolder, symbol Device:R_Small
- added R9: 0.1R, Resistor_SMD:R_0805_2012Metric_Pad1.20x1.40mm_HandSolder, symbol Device:R_Small
- added SW1: SW_SPDT, Button_Switch_SMD:SW_SPDT_PCM12, symbol Switch:SW_SPDT
- added TP1, TP2, TP3, TP4, TP5: TestPoint, TestPoint:TestPoint_Pad_D1.0mm, symbol Connector:TestPoint
- added U10: MT3608, Package_TO_SOT_SMD:SOT-23-6, symbol Regulator_Switching:MT3608
- added U2: DW01A, Package_TO_SOT_SMD:SOT-23-6, symbol Battery_Management:DW01A
- added U3: TP5100, Package_DFN_QFN:QFN-16-1EP_4x4mm_P0.65mm_EP2.1x2.1mm, symbol TP5100_BatCharg:TP5100
- added U4: AMS1117-3.3, Package_TO_SOT_SMD:SOT-223-3_TabPin2, symbol Regulator_Linear:AMS1117-3.3
Connections:
- net +3V3: now also C12.1, C14.1, R3.2, R4.2, TP5.1, U4.2 (VO)
- net +5V: now also C10.1, C11.1, C18.1, D4.1 (K), J1.2 (Pin_2), J1.6 (Pin_6), R18.2, TP4.1, U4.3 (VI); no longer U1.14 (5V)
- net GND: now also C10.2, C11.2, C12.2, C13.2, C14.2, C15.2, C17.2, C18.2, C3.2, C4.2, C5.2, C6.2, C9.2, D2.1 (K), D3.2 (A2), J1.4 (Pin_4), Q1.1 (D1), Q2.2 (S), R11.1, R12.1, R19.1, R2.1, R7.1, SW1.2 (B), U10.2 (GND), U3.12 (RTRICK), U3.17 (EP), U3.7 (GND), U4.1 (GND)
- net at U1.1 (PA02_A0_D0): now also R13.1
- net BTSENS: now reaches U1.2 (PA4_A1_D1)
- net BTSENS: now also C13.1, R6.1, R7.2
- net Heater_En: now reaches U1.4 (PA11_A3_D3)
- net Heater_En: now also R10.2
- net SDA: now reaches U1.5 (PA8_A4_D4_SDA)
- net SDA: now also J1.5 (Pin_5), R3.1
- net SCL: now reaches U1.6 (PA9_A5_D5_SCL)
- net SCL: now also J1.3 (Pin_3), R4.1
- new net: C17.1, L1.1, Q3.3 (D), R6.2, U10.4 (EN), U10.5 (IN)
- new net: D4.2 (A), L1.2, U10.1 (SW)
- new net: R2.2, U2.2 (CS)
- new net: R18.1, R19.2, U10.3 (FB)
- new net: TP1.1, U3.13 (CS)
- new net: J1.1 (Pin_1), Q2.3 (D)
- new net: C1.1, R1.2, U2.5 (VCC)
- new net: D1.2 (A), R5.1
- new net: D1.1 (K1), U3.15 (~{CHRG})
- new net: D1.3 (K2), U3.14 (~{STDBY})
- new net: R12.2, R8.1, U3.11 (TS)
- new net: Q3.1 (G), R14.1, SW1.1 (A)
- new net: BT1.2 (-), C1.2, Q1.3 (S2), U2.6 (GND)
- new net: Q2.1 (G), R10.1, R11.2
- new net: D2.2 (A), R13.2
- new net: L2.1, U3.2 (LX_1), U3.3 (LX_2)
- new net: C6.1, L2.2, R9.2, U3.8 (VS)
- new net: TP2.1, U3.6 (PWR_ON-)
- new net: Q1.2 (S1/D2), Q1.5 (S1/D2)
- new net: Q1.4 (G2), U2.1 (OD)
- new net: Q1.6 (G1), U2.3 (OC)
- new net +BATT: BT1.1 (+), C9.1, D3.1 (A1), Q3.2 (S), R1.1, R14.2, R9.1, TP3.1, U3.9 (BAT)
- new net VBUS: C15.1, C3.1, C4.1, R5.2, U1.14 (5V), U3.1 (VIN_1), U3.16 (VIN_4), U3.4 (VIN_2), U3.5 (VIN_3)
- new net VREG: C5.1, R8.2, U3.10 (VREG)
- no-connect marks 0 -> 8
Other:
- note added: "Alternate part: DMG9926UDM"
- note added: "Battery charger"
- note added: "Battery protection"
- note added: "ESP32-S3 SeeedStudio"
- note added: "SFM3300-D"
- note added: "Voltage converter"
- moved on the sheet: U1

Commit message: PCB changes
Parts:
- added H1, H2: MountingHole, MountingHole:MountingHole_2.2mm_M2, symbol Mechanical:MountingHole
Changed lines of the file:
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@@
+	)
+	(symbol
+		(lib_id "Mechanical:MountingHole")
+		(at 156.21 185.42 0)
+		(unit 1)
+		(exclude_from_sim no)
+		(in_bom no)
+		(on_board yes)
+		(dnp no)
+		(fields_autoplaced yes)
+		(property "Reference" "H2"
+			(at 158.75 184.1499 0)
+			(effects
+				(font
+					(size 1.27 1.27)
+				)
+				(justify left)
+			)
+		)
+		(property "Value" "MountingHole"
+			(at 158.75 186.6899 0)
+			(effects
+				(font
+					(size 1.27 1.27)
+				)
+				(justify left)
+			)
+		)
+		(property "Footprint" "MountingHole:MountingHole_2.2mm_M2"
+			(at 156.21 185.42 0)
+			(effects
+				(font
+					(size 1.27 1.27)
+				)
+				(hide yes)
+			)
+		)
+		(property "Datasheet" "~"
+			(at 156.21 185.42 0)
+			(effects
+				(font
+					(size 1.27 1.27)
+				)
+				(hide yes)
+			)
+		)
+		(property "Description" "Mounting Hole without connection"
+			(at 156.21 185.42 0)
+			(effects
+				(font
+					(size 1.27 1.27)
+				)
+				(hide yes)
+			)
+		)
+		(instances
+			(project "Vitalung_V0.1"
+				(path "/b803f8fb-0117-4d6e-9f54-ad7c3a060d4e"
+					(reference "H2")
+					(unit 1)
+				)
+			)
+		)
 	)
 	(symbol
@@
 					(unit 1)
 				)
+			)
+		)
+	)
+	(symbol
+		(lib_id "Mechanical:MountingHole")
+		(at 156.21 179.07 0)
+		(unit 1)
+		(exclude_from_sim no)
+		(in_bom no)
+		(on_board yes)
+		(dnp no)
+		(fields_autoplaced yes)
+		(property "Reference" "H1"
+			(at 158.75 177.7999 0)
+			(effects
+				(font
+					(size 1.27 1.27)
+				)
+				(justify left)
+			)
+		)
+		(property "Value" "MountingHole"
+			(at 158.75 180.3399 0)
+			(effects
+				(font
+					(size 1.27 1.27)
+				)
+				(justify left)
+			)
+		)
+		(property "Footprint" "MountingHole:MountingHole_2.2mm_M2"
+			(at 156.21 179.07 0)
+			(effects
+				(font
+					(size 1.27 1.27)
+				)
+				(hide yes)
+			)
+		)
+		(property "Datasheet" "~"
+			(at 156.21 179.07 0)
+			(effects
+				(font
+					(size 1.27 1.27)
+				)
+				(hide yes)
+			)
+		)
+		(property "Description" "Mounting Hole without connection"
+			(at 156.21 179.07 0)
+			(effects
+				(font
+					(size 1.27 1.27)
+				)
+				(hide yes)
+			)
+		)
+		(instances
+			(project ""
+				(path "/b803f8fb-0117-4d6e-9f54-ad7c3a060d4e"
+					(reference "H1")
+					(unit 1)
+				)

Commit message: PCB DXF change
Parts:
- removed Q3: AO3401A, Package_TO_SOT_SMD:SOT-23, symbol Transistor_FET:AO3401A
- removed R14: 100K, Resistor_SMD:R_0603_1608Metric_Pad0.98x0.95mm_HandSolder, symbol Device:R_Small
- added H3, H4: MountingHole, MountingHole:MountingHole_2.2mm_M2, symbol Mechanical:MountingHole
- SW1: footprint Button_Switch_SMD:SW_SPDT_PCM12 -> Button_Switch_THT:SW_Slide_SPDT_Angled_CK_OS102011MA1Q
Connections:
- net +BATT: now also SW1.2 (B)
- net GND: no longer SW1.2 (B)
- net Heater_En: now also U1.7 (PB08_A6_D6_TX); no longer U1.4 (PA11_A3_D3)
- net at C17.1, L1.1, R6.2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: now also SW1.1 (A)
- net at R13.1: now also U1.3 (PA10_A2_D2); no longer U1.1 (PA02_A0_D0)
Other:
- moved on the sheet: D2, H1, H2, R13, R3, R4, SW1

Commit message: Gerber generation
Parts:
- SW1: Robu_SKU R181035 -> (none)
- TP1, TP2, TP3, TP4, TP5: now left out of the parts list
Connections:
- net Red: now reaches D1.1 (K1), U3.15 (~{CHRG})
- net Green: now reaches D1.3 (K2), U3.14 (~{STDBY})
